Commit message: feat: add Noetic visual description release

File: urdf/b2arx_visual.urdf (robot description, URDF)
Before this commit: robot b2arx, 45 links, 44 joints
Links:
- link R5a: mass 0.42272 -> None; geometry visual mesh filename=package://b2arx_description/meshes/base_link.STL
- link R5a_link1: mass 0.096804 -> None; geometry visual mesh filename=package://b2arx_description/meshes/link1.STL
- link R5a_link2: mass 1.1988 -> None; geometry visual mesh filename=package://b2arx_description/meshes/link2.STL
- link R5a_link3: mass 0.84082 -> None; geometry visual mesh filename=package://b2arx_description/meshes/link3.STL
- link R5a_link4: mass 0.12432 -> None; geometry visual mesh filename=package://b2arx_description/meshes/link4.STL
- link R5a_link5: mass 0.63601 -> None; geometry visual mesh filename=package://b2arx_description/meshes/link5.STL
- link R5a_link6: mass 0.44089 -> None; geometry visual mesh filename=package://b2arx_description/meshes/link6.STL
- link R5a_link7: mass 0.064798 -> None; geometry visual mesh filename=package://b2arx_description/meshes/link7.STL
- link R5a_link8: mass 0.0647982 -> None; geometry visual mesh filename=package://b2arx_description/meshes/link8.STL
- link b2_description: mass 35.86 -> None; geometry visual mesh filename=package://b2arx_description/meshes/base_link.dae
- link b2_description_FL_calf: mass 0.404 -> None; geometry visual mesh filename=package://b2arx_description/meshes/FL_calf.dae
- link b2_description_FL_calf_rotor: mass 0.2734 -> None; geometry 
- link b2_description_FL_foot: mass 0.126 -> None; geometry 
- link b2_description_FL_hip: mass 2.673 -> None; geometry visual mesh filename=package://b2arx_description/meshes/FL_hip.dae
- link b2_description_FL_hip_rotor: mass 0.2734 -> None; geometry 
- link b2_description_FL_thigh: mass 4.536 -> None; geometry visual mesh filename=package://b2arx_description/meshes/FL_thigh.dae
- link b2_description_FL_thigh_rotor: mass 0.2734 -> None; geometry 
- link b2_description_FR_calf: mass 0.404 -> None; geometry visual mesh filename=package://b2arx_description/meshes/FR_calf.dae
- link b2_description_FR_calf_rotor: mass 0.2734 -> None; geometry 
- link b2_description_FR_foot: mass 0.126 -> None; geometry 
- link b2_description_FR_hip: mass 2.673 -> None; geometry visual mesh filename=package://b2arx_description/meshes/FR_hip.dae
- link b2_description_FR_hip_rotor: mass 0.2734 -> None; geometry 
- link b2_description_FR_thigh: mass 4.536 -> None; geometry visual mesh filename=package://b2arx_description/meshes/FR_thigh.dae
- link b2_description_FR_thigh_rotor: mass 0.2734 -> None; geometry 
- link b2_description_RL_calf: mass 0.404 -> None; geometry visual mesh filename=package://b2arx_description/meshes/RL_calf.dae
- link b2_description_RL_calf_rotor: mass 0.2734 -> None; geometry 
- link b2_description_RL_foot: mass 0.126 -> None; geometry 
- link b2_description_RL_hip: mass 2.673 -> None; geometry visual mesh filename=package://b2arx_description/meshes/RL_hip.dae
- link b2_description_RL_hip_rotor: mass 0.2734 -> None; geometry 
- link b2_description_RL_thigh: mass 4.536 -> None; geometry visual mesh filename=package://b2arx_description/meshes/RL_thigh.dae
- link b2_description_RL_thigh_rotor: mass 0.2734 -> None; geometry 
- link b2_description_RR_calf: mass 0.404 -> None; geometry visual mesh filename=package://b2arx_description/meshes/RR_calf.dae
- link b2_description_RR_calf_rotor: mass 0.2734 -> None; geometry 
- link b2_description_RR_foot: mass 0.126 -> None; geometry 
- link b2_description_RR_hip: mass 2.673 -> None; geometry visual mesh filename=package://b2arx_description/meshes/RR_hip.dae
- link b2_description_RR_hip_rotor: mass 0.2734 -> None; geometry 
- link b2_description_RR_thigh: mass 4.536 -> None; geometry visual mesh filename=package://b2arx_description/meshes/RR_thigh.dae
- link b2_description_RR_thigh_rotor: mass 0.2734 -> None; geometry 
- link b2_description_f_dc_link: mass 0 -> None
- link b2_description_f_oc_link: mass 0 -> None
- link b2_description_head_Link: mass 3.6885 -> None; geometry 
- link b2_description_imu_link: mass 0 -> None
- link b2_description_r_dc_link: mass 0 -> None
- link b2_description_r_oc_link: mass 0 -> None
- link b2_description_tail_link: mass 0.795 -> None; geometry 
